File: Modulator/Modulator.sch (KiCad schematic (older format))
At the start: 17 parts

Commit message: Updated modulator
Parts:
- removed U?: ADL5385, symbol ADL5385
- added C? (x6): 0.1u, symbol C_Small
- added R?: 10k, symbol R
- added U?: ADL5385, symbol ADL5385
Connections:
- net +5V: now also C?.2, C?.2, C?.2, R?.1, U?.11 (VPS2), U?.23 (VPS3), U?.24 (VPS3), U?.8 (VPS1), U?.9 (VPS1); no longer U?.1 (PD), U?.5 (PD)
- net GND: now also C?.1, C?.1, C?.1, U?.1 (NC), U?.15 (COM2), U?.16 (COM2), U?.19 (COM3), U?.2 (NC), U?.20 (COM3), U?.3 (NC), U?.4 (COM1), U?.5 (COM1), U?.6 (COM1), U?.PAD (GND)
- net I_n: now also U?.14 (IBB_n)
- net I_p: now also U?.13 (IBB_p)
- net Q_n: now also U?.17 (QBB_n)
- net Q_p: now also U?.18 (QBB_p)
- new net: C?.1, U?.21 (LOI_p)
- new net: C?.1, U?.22 (LOI_n)
- new net: C?.2, U?.7 (VOUT)
- new net Tx_En: R?.2, U?.1 (PD), U?.12 (ENBL), U?.5 (PD)
Other:
- note added: "TODO: Pull down to\ndisable Transmit\n"
- moved on the sheet: R?, RV?
