File: Subcircuits/Modulator/Modulator.sch (KiCad schematic (older format))
At the start: 24 parts

Commit message: Cleaned up components library
Parts:
- added JP? (x4): Jumper_NO_Small, symbol Jumper_NO_Small
- R? (x4): value 1k -> 2k
- RV? (x4): value 2k -> 5k
Changed lines of the file:
@@
 P 4025 2950
 F 0 "R?" V 3925 2950 50  0000 C CNN
-F 1 "1k" V 4025 2950 50  0000 C CNN
+F 1 "2k" V 4025 2950 50  0000 C CNN
 F 2 "" V 3955 2950 30  0000 C CNN
 F 3 "" H 4025 2950 30  0000 C CNN
@@
 P 4000 2650
 F 0 "R?" V 3900 2650 50  0000 C CNN
-F 1 "1k" V 4000 2650 50  0000 C CNN
+F 1 "2k" V 4000 2650 50  0000 C CNN
 F 2 "" V 3930 2650 30  0000 C CNN
 F 3 "" H 4000 2650 30  0000 C CNN
@@
 P 4000 4000
 F 0 "R?" V 3900 4000 50  0000 C CNN
-F 1 "1k" V 4000 4000 50  0000 C CNN
+F 1 "2k" V 4000 4000 50  0000 C CNN
 F 2 "" V 3930 4000 30  0000 C CNN
 F 3 "" H 4000 4000 30  0000 C CNN
@@
 P 4025 1600
 F 0 "R?" V 3925 1600 50  0000 C CNN
-F 1 "1k" V 4025 1600 50  0000 C CNN
+F 1 "2k" V 4025 1600 50  0000 C CNN
 F 2 "" V 3955 1600 30  0000 C CNN
 F 3 "" H 4025 1600 30  0000 C CNN
@@
 P 2675 1775
 F 0 "RV?" H 2675 1675 50  0000 C CNN
-F 1 "2k" H 2675 1775 50  0000 C CNN
+F 1 "5k" H 2675 1775 50  0000 C CNN
 F 2 "" H 2675 1775 60  0000 C CNN
 F 3 "" H 2675 1775 60  0000 C CNN
@@
 P 2550 2175
 F 0 "RV?" H 2550 2075 50  0000 C CNN
-F 1 "2k" H 2550 2175 50  0000 C CNN
+F 1 "5k" H 2550 2175 50  0000 C CNN
 F 2 "" H 2550 2175 60  0000 C CNN
 F 3 "" H 2550 2175 60  0000 C CNN
@@
 P 2675 3125
 F 0 "RV?" H 2675 3025 50  0000 C CNN
-F 1 "2k" H 2675 3125 50  0000 C CNN
+F 1 "5k" H 2675 3125 50  0000 C CNN
 F 2 "" H 2675 3125 60  0000 C CNN
 F 3 "" H 2675 3125 60  0000 C CNN
@@
 P 2550 3525
 F 0 "RV?" H 2550 3425 50  0000 C CNN
-F 1 "2k" H 2550 3525 50  0000 C CNN
+F 1 "5k" H 2550 3525 50  0000 C CNN
 F 2 "" H 2550 3525 60  0000 C CNN
 F 3 "" H 2550 3525 60  0000 C CNN
@@
 Text Notes 2350 1500 0    60   ~ 0
 Vocm 0.5V\nVref 3.3/2 = 1.65
-Text GLabel 4300 1975 2    60   Output ~ 0
+Text GLabel 4500 1975 2    60   Output ~ 0
 Q_p
-Text GLabel 4300 2125 2    60   Output ~ 0
+Text GLabel 4500 2125 2    60   Output ~ 0
 Q_n
-Text GLabel 4300 3325 2    60   Output ~ 0
+Text GLabel 4500 3325 2    60   Output ~ 0
 I_p
-Text GLabel 4300 3475 2    60   Output ~ 0
+Text GLabel 4500 3475 2    60   Output ~ 0
 I_n
 Text GLabel 7750 1650 1    60   Input ~ 0
@@
 Text Notes 4575 1525 0    60   ~ 0
 TODO: Pull down to\ndisable Transmit\n
+$Comp
+L Jumper_NO_Small JP?
+U 1 1 55FCE9C1
+P 4400 1975
+F 0 "JP?" H 4400 2055 50  0000 C CNN
+F 1 "Jumper_NO_Small" H 4410 1915 50  0001 C CNN
+F 2 "" H 4400 1975 60  0000 C CNN
+F 3 "" H 4400 1975 60  0000 C CNN
+	1    4400 1975
+	1    0    0    -1
+$EndComp
+$Comp
+L Jumper_NO_Small JP?
+U 1 1 55FCEA5F
+P 4400 2125
+F 0 "JP?" H 4400 2205 50  0000 C CNN
+F 1 "Jumper_NO_Small" H 4410 2065 50  0001 C CNN
+F 2 "" H 4400 2125 60  0000 C CNN
+F 3 "" H 4400 2125 60  0000 C CNN
+	1    4400 2125
+	1    0    0    -1
+$EndComp
+$Comp
+L Jumper_NO_Small JP?
+U 1 1 55FCEACB
+P 4400 3325
+F 0 "JP?" H 4400 3405 50  0000 C CNN
+F 1 "Jumper_NO_Small" H 4410 3265 50  0001 C CNN
+F 2 "" H 4400 3325 60  0000 C CNN
+F 3 "" H 4400 3325 60  0000 C CNN
+	1    4400 3325
+	1    0    0    -1
+$EndComp
+$Comp
+L Jumper_NO_Small JP?
+U 1 1 55FCEB68
+P 4400 3475
+F 0 "JP?" H 4400 3555 50  0000 C CNN
+F 1 "Jumper_NO_Small" H 4410 3415 50  0001 C CNN
+F 2 "" H 4400 3475 60  0000 C CNN
+F 3 "" H 4400 3475 60  0000 C CNN
+	1    4400 3475
+	1    0    0    -1
+$EndComp
 $EndSCHEMATC

Commit message: Updated Schematic
Parts:
- removed C? (x2): 0.22u, symbol C_Small
- removed C?: 0.1u, symbol C_Small
- removed JP? (x2): Jumper_NO_Small, symbol Jumper_NO_Small
- removed R? (x4): 2k, symbol R
- removed RV? (x4): 5k, symbol POT
- removed U? (x2): THS4532, symbol THS4532
- added C? (x2): 0.1u, symbol C_Small
- added JP? (x5): Jumper_NO_Small, symbol Jumper_NO_Small
- added R? (x8): 2.2k, symbol R
- added R? (x2): 10k, symbol R
- added RV? (x2): 20k, symbol POT
- added U? (x4): LMV324, symbol LMV324
- added U?: ADR130, symbol ADR130
Connections:
- net labels removed: Vocm
- wire segments 94 -> 100
- no-connect marks 4 -> 2
Other:
- note removed: "Vocm 0.5V\nVref 3.3/2 = 1.65"
- moved on the sheet: C?, P?

Commit message: More modifications to the schematics
Parts:
- added C? (x3): 1u, symbol C_Small
- added C?: 6.77n, symbol C
- added C?: 32.7n, symbol C
- added C? (x3): 10p, symbol C_Small
- added C? (x3): 0.1u, symbol C_Small
- added R?: 5.1k, symbol R
- added R?: 11.8k, symbol R
- added U?: ADF4351, symbol ADF4351
Connections:
- net labels added: +3.3V, PLLClkIn, PLLDataIn, PLLLe, PLLLock, PLLMuxOut, PLLOut_n, PLLOut_p
- wire segments 100 -> 146
- no-connect marks 2 -> 5
Other:
- moved on the sheet: C?, R?, U?

Commit message: Moar schematics!
Parts:
- removed P?: CONN_01X02, symbol CONN_01X02
- added C? (x6): 10p, symbol C_Small
- added C? (x6): 0.1u, symbol C_Small
- added C? (x4): 1u, symbol C_Small
- added P?: CONN_01X06, symbol CONN_01X06
- added P?: SMA, symbol BNC
- added P?: CONN_01X02, symbol CONN_01X02
- added R? (x2): 50, symbol R_Small
- added R? (x2): 20k, symbol R_Small
- added R? (x2): 2k, symbol R_Small
- added R? (x2): 4k, symbol R_Small
- added U? (x2): LTC1569-7, symbol LTC1569-7
- added W? (x10): TP, symbol TP
- added X?: ASTX-H11, symbol ASTX-H11
- C? (x2): value 0.1u -> 100p
Connections:
- wire segments 146 -> 275
- no-connect marks 5 -> 6
Other:
- note added: "Pull up over 1.5v\nto enable Transmit\n"
- note removed: "TODO: Pull down to\ndisable Transmit\n"
- moved on the sheet: C?, P?, R?, RV?, U?

Commit message: Made IQ LPF cutoff adjustable
Parts:
- removed C? (x2): 1u, symbol C_Small
- removed P?: CONN_01X02, symbol CONN_01X02
- removed R? (x2): 20k, symbol R_Small
- removed R?: 2k, symbol R_Small
- removed R?: 4k, symbol R_Small
- removed RV?: 20k, symbol POT
- removed U?: LTC1569-7, symbol LTC1569-7
- added C? (x2): 1u, symbol C_Small
- added P?: CONN_01X02, symbol CONN_01X02
- added R? (x2): 5k, symbol R_Small
- added R?: 2k, symbol R_Small
- added R?: 4k, symbol R_Small
- added RV? (x3): 20k, symbol POT
- added U?: LTC1569-7, symbol LTC1569-7
Connections:
- wire segments 275 -> 198
- no-connect marks 6 -> 8
Other:
- moved on the sheet: C?, RV?

Commit message: Finished modulator schematic
Parts:
- removed R?: 2k, symbol R_Small
- removed R?: 4k, symbol R_Small
- added C10: 10u, Capacitors_SMD:C_0805, symbol C_Small
- added C8: 1u, Capacitors_SMD:C_0805, symbol C_Small
- added C9: 100u, Capacitors_SMD:c_elec_6.3x5.8, symbol CP_Small
- added P3: CONN_01X02, Pin_Headers:Pin_Header_Straight_1x02, symbol CONN_01X02
- added U5: LD1117DT33TR, TO_SOT_Packages_SMD:TO-252-2Lead, symbol LD1117DT33TR
- C1, C11, C12, C13, C14, C15, C16, C17, C18, C19, C2, C20, C21, C22, C23, C24, C25, C26, C27, C28, C29, C3, C30, C31, C32, C33, C34, C35, C36, C37, C38, C39, C4, C5, C6, C7: renamed from C?; footprint (none) -> Capacitors_SMD:C_0805
- JP1, JP2, JP3, JP4, JP5, JP6, JP7: renamed from JP?; footprint (none) -> Footprints:SolderJump
- P1, P2: renamed from P?; footprint (none) -> Pin_Headers:Pin_Header_Straight_1x02
- P4: renamed from P?; footprint (none) -> Footprints:SMA-1814832
- P5: renamed from P?; footprint (none) -> Pin_Headers:Pin_Header_Straight_1x06
- R1: renamed from R?; value 4k -> 2.49k; footprint (none) -> Resistors_SMD:R_0805
- R10, R11, R12, R13, R14, R15, R16, R17, R18, R19, R3, R4, R5, R6, R7, R8, R9: renamed from R?; footprint (none) -> Resistors_SMD:R_0805
- R2: renamed from R?; value 2k -> 1.65k; footprint (none) -> Resistors_SMD:R_0805
- RV1, RV2, RV3, RV4: renamed from RV?; footprint (none) -> Footprints:PV36W
- U1, U2: renamed from U?; footprint (none) -> Housings_SOIC:SOIC-8_3.9x4.9mm_Pitch1.27mm
- U3: renamed from U?; footprint (none) -> TO_SOT_Packages_SMD:SOT-23-6
- U4: renamed from U?; footprint (none) -> Housings_SSOP:TSSOP-14_4.4x5mm_Pitch0.65mm
- U6: renamed from U?; footprint (none) -> Housings_DFN_QFN:QFN-32-1EP_5x5mm_Pitch0.5mm
- U7: renamed from U?; footprint (none) -> Housings_DFN_QFN:QFN-24-1EP_4x4mm_Pitch0.5mm
- W1, W10, W2, W3, W4, W5, W6, W7, W8, W9: renamed from W?; footprint (none) -> Measurement_Points:Measurement_Point_Round-SMD-Pad_Big
- X1: renamed from X?; footprint (none) -> Footprints:ASTX-H11
Connections:
- wire segments 198 -> 219
Other:
- moved on the sheet: C30, C32

Commit message: Annotated and PDFed modulator schematic
Other:
- note added: "10th order LPF with \nRRC impulse response"
- note added: "3.3V LDO"
- note added: "Bias Reference"
- note added: "Biasing and differential of I/Q"
- note added: "IQ Modulator"
- note added: "LO (Direct Conversion)"
- moved on the sheet: C11, C12, C13, C14, C15, C16, C17, C18, C19, C20, C21, C23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

Commit message: Finished prototype modulator board
Parts:
- removed P1, P2: CONN_01X02, Pin_Headers:Pin_Header_Straight_1x02, symbol CONN_01X02
- removed W2, W3, W4, W5, W6, W9: TP, Measurement_Points:Measurement_Point_Round-SMD-Pad_Big, symbol TP
- added P1: CONN_01X03, Pin_Headers:Pin_Header_Straight_1x03, symbol CONN_01X03
- W1: footprint Measurement_Points:Measurement_Point_Round-SMD-Pad_Big -> Measurement_Points:Measurement_Point_Round-SMD-Pad_Small
- W2: renamed from W7; footprint Measurement_Points:Measurement_Point_Round-SMD-Pad_Big -> Measurement_Points:Measurement_Point_Round-SMD-Pad_Small
- W3: renamed from W8; footprint Measurement_Points:Measurement_Point_Round-SMD-Pad_Big -> Measurement_Points:Measurement_Point_Round-SMD-Pad_Small
- W5: renamed from W10; footprint Measurement_Points:Measurement_Point_Round-SMD-Pad_Big -> Measurement_Points:Measurement_Point_Round-SMD-Pad_Small
- renumbered C12 to C11, C13 to C12, C11 to C13, C21 to C19, C19 to C20, C23 to C21, C20 to C22, C25 to C23, C29 to C24, C24 to C25, C22 to C26, C26 to C27, C31 to C28, C27 to C29, C33 to C31, C28 to C32, C32 to C33, P3 to P2, P4 to P3, P5 to P4
Connections:
- net labels added: I_N, I_P, PLLOut_N, PLLOut_P, PLL_N, PLL_P, Q_N, Q_P, pI_N, pI_P, pQ_N, pQ_P
- net labels removed: I_n, I_p, PLLOut_n, PLLOut_p, Q_n, Q_p
Other:
- moved on the sheet: C11, C12
